Commit message: updated urdf description

File: description/robot_description.xacro (robot description, xacro)
@@ -1,4 +1,5 @@
 <?xml version = "1.0"?>
-<robot name = "scara" >
+<robot xmlns:xacro="http://www.ros.org/wiki/xacro" name="robot">
+    <xacro:include filename="ros2_control.xacro" />
     <link name="world"/>
     <joint name="fixed" type="fixed">
@@ -9,5 +10,5 @@
         <visual>
             <geometry>
-                <mesh filename = "package://scara_robot_description/meshes/base.stl" scale = "1 1 1"/>
+                <mesh filename = "file://$(find scara_robot_description)/meshes/base.stl" scale = "1 1 1"/>
             </geometry>
             <origin rpy = "0 0 0" xyz = "0 0 0"/>
@@ -15,5 +16,5 @@
         <collision>
             <geometry>
-                <mesh filename = "package://scara_robot_description/meshes/base_low.stl" scale = "1 1 1"/>
+                <mesh filename = "file://$(find scara_robot_description)/meshes/base_low.stl" scale = "1 1 1"/>
             </geometry>
             <origin rpy = "0 0 0" xyz = "0 0 0"/>
@@ -32,19 +33,8 @@
         <limit effort = "10" lower = "-3.14" upper = "3.14" velocity = "0.5" />
     </joint>
-    <!--TRANSMISSION-->
-    <transmission name = "base_link_brazo_trans">
-        <type>transmission_interface/SimpleTransmission</type>
-        <joint name="base_link_link_01">
-            <hardwareInterface>hardware_interface/EffortJointInterface</hardwareInterface>
-        </joint>
-        <actuator name="base_link_link_01">
-            <hardwareInterface>hardware_interface/EffortJointInterface</hardwareInterface>
-            <mechanicalReduction>1</mechanicalReduction>
-        </actuator>
-    </transmission>
     <link name = "link_01">
         <visual>
             <geometry>
-                <mesh filename = "package://scara_robot_description/meshes/brazo.stl" scale = "1 1 1"/>
+                <mesh filename = "file://$(find scara_robot_description)/meshes/brazo.stl" scale = "1 1 1"/>
             </geometry>
             <origin rpy = "0 0 0" xyz = "0 0 0"/>
@@ -52,5 +42,5 @@
         <collision>
             <geometry>
-                <mesh filename = "package://scara_robot_description/meshes/brazo_low.stl" scale = "1 1 1"/>
+                <mesh filename = "file://$(find scara_robot_description)/meshes/brazo_low.stl" scale = "1 1 1"/>
             </geometry>
             <origin rpy = "0 0 0" xyz = "0 0 0"/>
@@ -69,19 +59,8 @@
         <limit effort = "10" lower = "-3.14" upper = "3.14" velocity = "0.5" />
     </joint>
-    <!--TRANSMISSION-->
-    <transmission name = "link_01_brazo_2_trans">
-        <type>transmission_interface/SimpleTransmission</type>
-        <joint name="link_01_link_02">
-            <hardwareInterface>hardware_interface/EffortJointInterface</hardwareInterface>
-        </joint>
-        <actuator name="link_01_link_02">
-            <hardwareInterface>hardware_interface/EffortJointInterface</hardwareInterface>
-            <mechanicalReduction>1</mechanicalReduction>
-        </actuator>
-    </transmission>
     <link name = "link_02">
         <visual>
             <geometry>
-                <mesh filename = "package://scara_robot_description/meshes/brazo_2.stl" scale = "1 1 1"/>
+                <mesh filename = "file://$(find scara_robot_description)/meshes/brazo_2.stl" scale = "1 1 1"/>
             </geometry>
             <origin rpy = "0 0 0" xyz = "0 0 0"/>
@@ -89,5 +68,5 @@
         <collision>
             <geometry>
-                <mesh filename = "package://scara_robot_description/meshes/brazo_low_2.stl" scale = "1 1 1"/>
+                <mesh filename = "file://$(find scara_robot_description)/meshes/brazo_low_2.stl" scale = "1 1 1"/>
             </geometry>
             <origin rpy = "0 0 0" xyz = "0 0 0"/>
@@ -106,19 +85,8 @@
         <limit effort = "100" lower = "-0.15" upper = "0.0" velocity = "0.5" />
     </joint>
-    <!--TRANSMISSION-->
-    <transmission name = "link_02_link_03_trans">
-        <type>transmission_interface/SimpleTransmission</type>
-        <joint name="link_02_link_03">
-            <hardwareInterface>hardware_interface/EffortJointInterface</hardwareInterface>
-        </joint>
-        <actuator name="link_02_link_03">
-            <hardwareInterface>hardware_interface/EffortJointInterface</hardwareInterface>
-            <mechanicalReduction>1</mechanicalReduction>
-        </actuator>
-    </transmission>
     <link name = "link_03">
         <visual>
             <geometry>
-                <mesh filename = "package://scara_robot_description/meshes/lineal.stl" scale = "1 1 1"/>
+                <mesh filename = "file://$(find scara_robot_description)/meshes/lineal.stl" scale = "1 1 1"/>
             </geometry>
             <origin rpy = "0 0 0" xyz = "0 0 0"/>
@@ -126,5 +94,5 @@
         <collision>
             <geometry>
-                <mesh filename = "package://scara_robot_description/meshes/lineal.stl" scale = "1 1 1"/>
+                <mesh filename = "file://$(find scara_robot_description)/meshes/lineal.stl" scale = "1 1 1"/>
             </geometry>
             <origin rpy = "0 0 0" xyz = "0 0 0"/>
@@ -136,8 +104,3 @@
         </inertial>
     </link>
-    <gazebo>
-        <plugin name = "gazebo_ros_control" filename = "libgazebo_ros_control.so">
-            <robotNamespace>/scara</robotNamespace>
-        </plugin>
-    </gazebo>
 </robot>

Commit message: changed collisions models

File: description/robot_description.xacro (robot description, xacro)
@@ -19,5 +19,5 @@
         <collision>
             <geometry>
-                <mesh filename = "file://$(find scara_robot_description)/meshes/base_low.stl" scale = "1 1 1"/>
+                <mesh filename = "file://$(find scara_robot_description)/meshes/base.stl" scale = "1 1 1"/>
             </geometry>
             <origin rpy = "0 0 0" xyz = "0 0 0"/>
@@ -45,5 +45,5 @@
         <collision>
             <geometry>
-                <mesh filename = "file://$(find scara_robot_description)/meshes/brazo_low.stl" scale = "1 1 1"/>
+                <mesh filename = "file://$(find scara_robot_description)/meshes/brazo.stl" scale = "1 1 1"/>
             </geometry>
             <origin rpy = "0 0 0" xyz = "0 0 0"/>
@@ -71,5 +71,5 @@
         <collision>
             <geometry>
-                <mesh filename = "file://$(find scara_robot_description)/meshes/brazo_low_2.stl" scale = "1 1 1"/>
+                <mesh filename = "file://$(find scara_robot_description)/meshes/brazo_2.stl" scale = "1 1 1"/>
             </geometry>
             <origin rpy = "0 0 0" xyz = "0 0 0"/>
